File: tuer-steuerung/tuer-steuerungEvolved/motor.sch (KiCad schematic (older format))
At the start: 9 parts

Commit message: Imported updated requirements for new door pcb
Parts:
- IC?: symbol L6203:L6203 -> tuer-steuerungEvolved-rescue:L6203-L6203
Changed lines of the file:
@@
 EESchema Schematic File Version 4
-LIBS:tuer-steuerungEvolved-cache
-EELAYER 26 0
+EELAYER 30 0
 EELAYER END
 $Descr A4 11693 8268
@@
 $EndDescr
 $Comp
-L L6203:L6203 IC?
+L tuer-steuerungEvolved-rescue:L6203-L6203 IC?
 U 1 1 5BF1DEB4
 P 3600 2500
 AR Path="/5BF197FE/5BF1DEB4" Ref="IC?"  Part="1"
 AR Path="/5BF1DE2A/5BF1DEB4" Ref="IC?"  Part="1"
+AR Path="/5BF1DEB4" Ref="IC?"  Part="1"
 F 0 "IC?" H 3600 2550 50  0000 C CNN
 F 1 "L6203" H 3600 2400 50  0000 C CNN
